Commit message: tune values for zed camera

File: nerf_ws/src/zed_description/urdf/zed_descr.urdf.xacro (robot description, xacro)
@@ -26,5 +26,5 @@
   <xacro:arg name="cam_yaw"       default="0.0" />
   <xacro:arg name="gnss_frame"    default="" />
-  <xacro:include filename="$(find zed_wrapper)/urdf/zed_macro.urdf.xacro" />
+  <xacro:include filename="$(find zed_description)/urdf/zed_macro.urdf.xacro" />
   <xacro:zed_camera name="$(arg camera_name)" model="$(arg camera_model)" parent="$(arg base_frame)">
     <origin

File: nerf_ws/src/zed_description/urdf/zed_macro.urdf.xacro (robot description, xacro)
@@ -16,5 +16,5 @@
 -->
 <robot xmlns:xacro="http://wiki.ros.org/xacro">
-  <xacro:include filename="$(find zed_wrapper)/urdf/include/materials.urdf.xacro" />
+  <xacro:include filename="$(find zed_description)/urdf/include/materials.urdf.xacro" />
   <xacro:property name="M_PI"     value="3.1415926535897931" />
   <!--
@@ -105,5 +105,5 @@
       <parent link="${name}_april_tag"/>
       <child link="${parent}"/>
-      <origin xyz="-0.00682 -0.007682 0.029492" rpy="0.0 -3.115 -1.57" />
+      <origin xyz="-0.00682 -0.007682 0.029492" rpy="0.0 -3.11 -1.56" />
     </joint>
     <!-- Left Camera -->
